Commit message: Expand canonical golfer URDF generation and validation (#42)
* feat(model): expand canonical urdf export

* Fix CI/CD linting and testing issues in URDF exporter and validation tests

File: models/generated/golfer.urdf (robot description, URDF)
Before this commit: robot golfer, 1 links, 0 joints
Links:
- added link club_head, mass 0.2; visual box size=0.12 0.08 0.04
- added link club_shaft, mass 0.05; visual cylinder length=1.0 radius=0.015
- added link fingers_left, mass 0.2; visual box size=0.05 0.08 0.02
- added link fingers_right, mass 0.2; visual box size=0.05 0.08 0.02
- added link forearm_left, mass 1.18; visual cylinder length=0.26 radius=0.045
- added link forearm_left_intermediate, mass 0.001
- added link forearm_right, mass 1.18; visual cylinder length=0.26 radius=0.045
- added link forearm_right_intermediate, mass 0.001
- added link hand_left, mass 0.61; visual cylinder length=0.19 radius=0.04
- added link hand_left_intermediate, mass 0.001
- added link hand_right, mass 0.61; visual cylinder length=0.19 radius=0.04
- added link hand_right_intermediate, mass 0.001
- added link left_foot, mass 1.37; visual box size=0.26 0.1 0.07
- added link left_foot_intermediate, mass 0.001
- added link left_shank, mass 3.53; visual cylinder length=0.43 radius=0.05
- added link left_thigh, mass 7.05; visual cylinder length=0.43 radius=0.06
- added link left_thigh_gimbal_y, mass 0.001
- added link left_thigh_gimbal_z, mass 0.001
- added link left_toes, mass 0.3; visual box size=0.1 0.08 0.03
- added link lumbar1, mass 2.0; visual cylinder length=0.24 radius=0.08
- added link lumbar1_intermediate, mass 0.001
- added link lumbar2, mass 2.0; visual cylinder length=0.24 radius=0.08
- added link lumbar2_intermediate, mass 0.001
- added link lumbar3, mass 2.0; visual cylinder length=0.24 radius=0.08
- added link lumbar3_intermediate, mass 0.001
- added link right_foot, mass 1.37; visual box size=0.26 0.1 0.07
- added link right_foot_intermediate, mass 0.001
- added link right_shank, mass 3.53; visual cylinder length=0.43 radius=0.05
- added link right_thigh, mass 7.05; visual cylinder length=0.43 radius=0.06
- added link right_thigh_gimbal_y, mass 0.001
- added link right_thigh_gimbal_z, mass 0.001
- added link right_toes, mass 0.3; visual box size=0.1 0.08 0.03
- added link scapula_left, mass 1.5; visual box size=0.12 0.08 0.05
- added link scapula_left_intermediate, mass 0.001
- added link scapula_right, mass 1.5; visual box size=0.12 0.08 0.05
- added link scapula_right_intermediate, mass 0.001
- added link thorax1, mass 1.5; visual cylinder length=0.2 radius=0.08
- added link thorax2, mass 1.5; visual cylinder length=0.2 radius=0.08
- added link thorax3, mass 1.5; visual cylinder length=0.2 radius=0.08
- added link upper_arm_left, mass 1.98; visual cylinder length=0.28 radius=0.05
- added link upper_arm_left_gimbal_y, mass 0.001
- added link upper_arm_left_gimbal_z, mass 0.001
- added link upper_arm_right, mass 1.98; visual cylinder length=0.28 radius=0.05
- added link upper_arm_right_gimbal_y, mass 0.001
- added link upper_arm_right_gimbal_z, mass 0.001
- link pelvis: mass 11.70 -> 11.7; geometry visual cylinder length=0.4 radius=0.15
Joints:
- added joint club_shaft_to_club_head: type fixed, parent club_shaft, child club_head, origin xyz=0.0 0.0 -0.5 rpy=0.0 0.0 0.0
- added joint forearm_left_intermediate_to_forearm_left: type revolute, parent forearm_left_intermediate, child forearm_left, origin xyz=0.0 0.0 0.0 rpy=0.0 0.0 0.0, axis 1 0 0, limit lower=-1.57 upper=1.57 effort=1000.0 velocity=10.0
- added joint forearm_left_to_hand_left_intermediate: type revolute, parent forearm_left, child hand_left_intermediate, origin xyz=0.0 0.0 -0.19 rpy=0.0 0.0 0.0, axis 0 1 0, limit lower=-1.22 upper=1.22 effort=1000.0 velocity=10.0
- added joint forearm_right_intermediate_to_forearm_right: type revolute, parent forearm_right_intermediate, child forearm_right, origin xyz=0.0 0.0 0.0 rpy=0.0 0.0 0.0, axis 1 0 0, limit lower=-1.57 upper=1.57 effort=1000.0 velocity=10.0
- added joint forearm_right_to_hand_right_intermediate: type revolute, parent forearm_right, child hand_right_intermediate, origin xyz=0.0 0.0 -0.19 rpy=0.0 0.0 0.0, axis 0 1 0, limit lower=-1.22 upper=1.22 effort=1000.0 velocity=10.0
- added joint hand_left_intermediate_to_hand_left: type revolute, parent hand_left_intermediate, child hand_left, origin xyz=0.0 0.0 0.0 rpy=0.0 0.0 0.0, axis 0 0 1, limit lower=-0.52 upper=0.7 effort=1000.0 velocity=10.0
- added joint hand_left_to_club_shaft: type fixed, parent hand_left, child club_shaft, origin xyz=0.0 0.0 -0.12 rpy=0.0 0.0 0.0
- added joint hand_left_to_fingers_left: type revolute, parent hand_left, child fingers_left, origin xyz=0.0 0.0 -0.05 rpy=0.0 0.0 0.0, axis 0 1 0, limit lower=0.0 upper=1.57 effort=1000.0 velocity=10.0
- added joint hand_right_intermediate_to_hand_right: type revolute, parent hand_right_intermediate, child hand_right, origin xyz=0.0 0.0 0.0 rpy=0.0 0.0 0.0, axis 0 0 1, limit lower=-0.52 upper=0.7 effort=1000.0 velocity=10.0
- added joint hand_right_to_fingers_right: type revolute, parent hand_right, child fingers_right, origin xyz=0.0 0.0 -0.05 rpy=0.0 0.0 0.0, axis 0 1 0, limit lower=0.0 upper=1.57 effort=1000.0 velocity=10.0
- added joint left_foot_intermediate_to_left_foot: type revolute, parent left_foot_intermediate, child left_foot, origin xyz=0.0 0.0 0.0 rpy=0.0 0.0 0.0, axis 0 1 0, limit lower=-0.35 upper=0.35 effort=1000.0 velocity=10.0
- added joint left_foot_to_left_toes: type revolute, parent left_foot, child left_toes, origin xyz=0.12 0.0 -0.02 rpy=0.0 0.0 0.0, axis 0 1 0, limit lower=-0.35 upper=0.52 effort=1000.0 velocity=10.0
- added joint left_shank_to_left_foot_intermediate: type revolute, parent left_shank, child left_foot_intermediate, origin xyz=0.0 0.0 -0.43 rpy=0.0 0.0 0.0, axis 1 0 0, limit lower=-0.7 upper=0.52 effort=1000.0 velocity=10.0
- added joint left_thigh_gimbal_y_to_left_thigh: type revolute, parent left_thigh_gimbal_y, child left_thigh, origin xyz=0.0 0.0 0.0 rpy=0.0 0.0 0.0, axis 0 0 1, limit lower=-0.7 upper=0.7 effort=1000.0 velocity=10.0
- added joint left_thigh_gimbal_z_to_left_thigh_gimbal_y: type revolute, parent left_thigh_gimbal_z, child left_thigh_gimbal_y, origin xyz=0.0 0.0 0.0 rpy=0.0 0.0 0.0, axis 1 0 0, limit lower=-0.87 upper=0.52 effort=1000.0 velocity=10.0
- added joint left_thigh_to_left_shank: type revolute, parent left_thigh, child left_shank, origin xyz=0.0 0.0 -0.43 rpy=0.0 0.0 0.0, axis 0 1 0, limit lower=0.0 upper=2.62 effort=1000.0 velocity=10.0
- added joint lumbar1_intermediate_to_lumbar1: type revolute, parent lumbar1_intermediate, child lumbar1, origin xyz=0.0 0.0 0.0 rpy=0.0 0.0 0.0, axis 0 1 0, limit lower=-0.35 upper=0.35 effort=1000.0 velocity=10.0
- added joint lumbar1_to_lumbar2_intermediate: type revolute, parent lumbar1, child lumbar2_intermediate, origin xyz=0.0 0.0 0.12 rpy=0.0 0.0 0.0, axis 1 0 0, limit lower=-0.7 upper=0.52 effort=1000.0 velocity=10.0
- added joint lumbar2_intermediate_to_lumbar2: type revolute, parent lumbar2_intermediate, child lumbar2, origin xyz=0.0 0.0 0.0 rpy=0.0 0.0 0.0, axis 0 1 0, limit lower=-0.35 upper=0.35 effort=1000.0 velocity=10.0
- added joint lumbar2_to_lumbar3_intermediate: type revolute, parent lumbar2, child lumbar3_intermediate, origin xyz=0.0 0.0 0.12 rpy=0.0 0.0 0.0, axis 1 0 0, limit lower=-0.7 upper=0.52 effort=1000.0 velocity=10.0
- added joint lumbar3_intermediate_to_lumbar3: type revolute, parent lumbar3_intermediate, child lumbar3, origin xyz=0.0 0.0 0.0 rpy=0.0 0.0 0.0, axis 0 1 0, limit lower=-0.35 upper=0.35 effort=1000.0 velocity=10.0
- added joint lumbar3_to_thorax1: type revolute, parent lumbar3, child thorax1, origin xyz=0.0 0.0 0.12 rpy=0.0 0.0 0.0, axis 0 0 1, limit lower=-1.0 upper=1.0 effort=1000.0 velocity=10.0
- added joint pelvis_to_left_thigh_gimbal_z: type revolute, parent pelvis, child left_thigh_gimbal_z, origin xyz=0.0 0.09 -0.05 rpy=0.0 0.0 0.0, axis 0 1 0, limit lower=-1.57 upper=1.57 effort=1000.0 velocity=10.0
- added joint pelvis_to_lumbar1_intermediate: type revolute, parent pelvis, child lumbar1_intermediate, origin xyz=0.0 0.0 0.12 rpy=0.0 0.0 0.0, axis 1 0 0, limit lower=-0.7 upper=0.52 effort=1000.0 velocity=10.0
- added joint pelvis_to_right_thigh_gimbal_z: type revolute, parent pelvis, child right_thigh_gimbal_z, origin xyz=0.0 -0.09 -0.05 rpy=0.0 0.0 0.0, axis 0 1 0, limit lower=-1.57 upper=1.57 effort=1000.0 velocity=10.0
- added joint right_foot_intermediate_to_right_foot: type revolute, parent right_foot_intermediate, child right_foot, origin xyz=0.0 0.0 0.0 rpy=0.0 0.0 0.0, axis 0 1 0, limit lower=-0.35 upper=0.35 effort=1000.0 velocity=10.0
- added joint right_foot_to_right_toes: type revolute, parent right_foot, child right_toes, origin xyz=0.12 0.0 -0.02 rpy=0.0 0.0 0.0, axis 0 1 0, limit lower=-0.35 upper=0.52 effort=1000.0 velocity=10.0
- added joint right_shank_to_right_foot_intermediate: type revolute, parent right_shank, child right_foot_intermediate, origin xyz=0.0 0.0 -0.43 rpy=0.0 0.0 0.0, axis 1 0 0, limit lower=-0.7 upper=0.52 effort=1000.0 velocity=10.0
- added joint right_thigh_gimbal_y_to_right_thigh: type revolute, parent right_thigh_gimbal_y, child right_thigh, origin xyz=0.0 0.0 0.0 rpy=0.0 0.0 0.0, axis 0 0 1, limit lower=-0.7 upper=0.7 effort=1000.0 velocity=10.0
- added joint right_thigh_gimbal_z_to_right_thigh_gimbal_y: type revolute, parent right_thigh_gimbal_z, child right_thigh_gimbal_y, origin xyz=0.0 0.0 0.0 rpy=0.0 0.0 0.0, axis 1 0 0, limit lower=-0.87 upper=0.52 effort=1000.0 velocity=10.0
- added joint right_thigh_to_right_shank: type revolute, parent right_thigh, child right_shank, origin xyz=0.0 0.0 -0.43 rpy=0.0 0.0 0.0, axis 0 1 0, limit lower=0.0 upper=2.62 effort=1000.0 velocity=10.0
- added joint scapula_left_intermediate_to_scapula_left: type revolute, parent scapula_left_intermediate, child scapula_left, origin xyz=0.0 0.0 0.0 rpy=0.0 0.0 0.0, axis 0 1 0, limit lower=-0.52 upper=0.52 effort=1000.0 velocity=10.0
- added joint scapula_left_to_upper_arm_left_gimbal_z: type revolute, parent scapula_left, child upper_arm_left_gimbal_z, origin xyz=0.0 0.04 0.1 rpy=0.0 0.0 0.0, axis 0 1 0, limit lower=-1.57 upper=3.1416 effort=1000.0 velocity=10.0
- added joint scapula_right_intermediate_to_scapula_right: type revolute, parent scapula_right_intermediate, child scapula_right, origin xyz=0.0 0.0 0.0 rpy=0.0 0.0 0.0, axis 0 1 0, limit lower=-0.52 upper=0.52 effort=1000.0 velocity=10.0
- added joint scapula_right_to_upper_arm_right_gimbal_z: type revolute, parent scapula_right, child upper_arm_right_gimbal_z, origin xyz=0.0 -0.04 0.1 rpy=0.0 0.0 0.0, axis 0 1 0, limit lower=-1.57 upper=3.1416 effort=1000.0 velocity=10.0
- added joint thorax1_to_thorax2: type revolute, parent thorax1, child thorax2, origin xyz=0.0 0.0 0.1 rpy=0.0 0.0 0.0, axis 0 0 1, limit lower=-1.0 upper=1.0 effort=1000.0 velocity=10.0
- added joint thorax2_to_thorax3: type revolute, parent thorax2, child thorax3, origin xyz=0.0 0.0 0.1 rpy=0.0 0.0 0.0, axis 0 0 1, limit lower=-1.0 upper=1.0 effort=1000.0 velocity=10.0
- added joint thorax3_to_scapula_left_intermediate: type revolute, parent thorax3, child scapula_left_intermediate, origin xyz=0.0 0.18 0.28 rpy=0.0 0.0 0.0, axis 0 0 1, limit lower=-0.35 upper=0.7 effort=1000.0 velocity=10.0
- added joint thorax3_to_scapula_right_intermediate: type revolute, parent thorax3, child scapula_right_intermediate, origin xyz=0.0 -0.18 0.28 rpy=0.0 0.0 0.0, axis 0 0 1, limit lower=-0.35 upper=0.7 effort=1000.0 velocity=10.0
- added joint upper_arm_left_gimbal_y_to_upper_arm_left: type revolute, parent upper_arm_left_gimbal_y, child upper_arm_left, origin xyz=0.0 0.0 0.0 rpy=0.0 0.0 0.0, axis 0 0 1, limit lower=-1.57 upper=1.57 effort=1000.0 velocity=10.0
- added joint upper_arm_left_gimbal_z_to_upper_arm_left_gimbal_y: type revolute, parent upper_arm_left_gimbal_z, child upper_arm_left_gimbal_y, origin xyz=0.0 0.0 0.0 rpy=0.0 0.0 0.0, axis 1 0 0, limit lower=-0.52 upper=2.09 effort=1000.0 velocity=10.0
- added joint upper_arm_left_to_forearm_left_intermediate: type revolute, parent upper_arm_left, child forearm_left_intermediate, origin xyz=0.0 0.0 -0.26 rpy=0.0 0.0 0.0, axis 0 1 0, limit lower=0.0 upper=2.62 effort=1000.0 velocity=10.0
- added joint upper_arm_right_gimbal_y_to_upper_arm_right: type revolute, parent upper_arm_right_gimbal_y, child upper_arm_right, origin xyz=0.0 0.0 0.0 rpy=0.0 0.0 0.0, axis 0 0 1, limit lower=-1.57 upper=1.57 effort=1000.0 velocity=10.0
- added joint upper_arm_right_gimbal_z_to_upper_arm_right_gimbal_y: type revolute, parent upper_arm_right_gimbal_z, child upper_arm_right_gimbal_y, origin xyz=0.0 0.0 0.0 rpy=0.0 0.0 0.0, axis 1 0 0, limit lower=-0.52 upper=2.09 effort=1000.0 velocity=10.0
- added joint upper_arm_right_to_forearm_right_intermediate: type revolute, parent upper_arm_right, child forearm_right_intermediate, origin xyz=0.0 0.0 -0.26 rpy=0.0 0.0 0.0, axis 0 1 0, limit lower=0.0 upper=2.62 effort=1000.0 velocity=10.0
